File: hardware/pcb/r3_senderEsp/r3_senderEsp.kicad_sch (KiCad schematic)
At the start: 17 parts, among them J1 RFID-RC522, J2 KY-021, J3 KY-021, J4 Links, J5 Rechts

Commit message: Add files via upload
Connections:
- net +5V: no longer J1.1 (Pin_1)
- net at A1.4 (3V3): now also J1.1 (Pin_1)
Changed lines of the file:
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@@
-	)
-	(junction
-		(at 114.3 27.94)
-		(diameter 0)
-		(color 0 0 0 0)
 	)
 	(junction
@@
 	(wire
 		(pts
-			(xy 114.3 27.94) (xy 88.9 27.94)
-		)
-		(stroke
-			(width 0)
-			(type default)
-			(color 253 0 3 1)
+			(xy 88.9 27.94) (xy 128.27 27.94)
+		)
+		(stroke
+			(width 0)
+			(type default)
+			(color 253 0 3 1)
+		)
+	)
+	(wire
+		(pts
+			(xy 191.77 38.1) (xy 191.77 40.64)
+		)
+		(stroke
+			(width 0)
+			(type default)
+			(color 172 0 0 1)
 		)
 	)
@@
 	(wire
 		(pts
-			(xy 114.3 27.94) (xy 114.3 96.52)
-		)
-		(stroke
-			(width 0)
-			(type default)
-			(color 253 0 3 1)
-		)
-	)
-	(wire
-		(pts
 			(xy 152.4 83.82) (xy 152.4 76.2)
 		)
@@
 	(wire
 		(pts
+			(xy 163.83 27.94) (xy 194.31 27.94)
+		)
+		(stroke
+			(width 0)
+			(type default)
+			(color 253 0 3 1)
+		)
+	)
+	(wire
+		(pts
 			(xy 176.53 66.04) (xy 161.29 66.04)
 		)
@@
 	(wire
 		(pts
+			(xy 114.3 38.1) (xy 191.77 38.1)
+		)
+		(stroke
+			(width 0)
+			(type default)
+			(color 172 0 0 1)
+		)
+	)
+	(wire
+		(pts
 			(xy 191.77 118.11) (xy 191.77 130.81)
 		)
@@
 	(wire
 		(pts
+			(xy 114.3 38.1) (xy 114.3 96.52)
+		)
+		(stroke
+			(width 0)
+			(type default)
+			(color 199 0 0 1)
+		)
+	)
+	(wire
+		(pts
 			(xy 88.9 27.94) (xy 88.9 52.07)
 		)
@@
 	(wire
 		(pts
-			(xy 114.3 27.94) (xy 128.27 27.94)
-		)
-		(stroke
-			(width 0)
-			(type default)
-			(color 253 0 3 1)
-		)
-	)
-	(wire
-		(pts
 			(xy 176.53 68.58) (xy 170.18 68.58)
 		)
@@
 		)
 	)
-	(wire
-		(pts
-			(xy 163.83 27.94) (xy 194.31 27.94)
-		)
-		(stroke
-			(width 0)
-			(type default)
-			(color 253 0 3 1)
-		)
-	)
